File: supplyboard/supplyboard.kicad_pcb (KiCad board)
At the start: 2 copper layers, 95 parts, among them J1 Screw_Terminal_01x03, J2 FEMALE 06, J3 Conn_01x02, Q1 MBR20100CT, Q2 MBR20100CT, Q3 PN2222A, Q4 IRF540N, Q5 PN2222A, T1 SM_FB, U1 EL817, U2 UC3843_DIP8, U3 TL431D, U4 L7805, U5 LM358N_NOPB, U6 LM2575-12BU

Commit message: finalgerber
Parts:
- added ?: , logo2:logo2, F.Cu at (160.0, 128.9)
- added ?: MountingHole_3.5mm, MountingHole:MountingHole_3.5mm, F.Cu at (121.3, 85.1)
- added ?: MountingHole_3.2mm_M3, MountingHole:MountingHole_3.2mm_M3, F.Cu at (186.4, 101.1)
- added ?: MountingHole_3.5mm, MountingHole:MountingHole_3.5mm, F.Cu at (42.0, 82.5)
- added ?: MountingHole_3.5mm, MountingHole:MountingHole_3.5mm, F.Cu at (189.7, 82.5)
- added ?: MountingHole_3.5mm, MountingHole:MountingHole_3.5mm, F.Cu at (189.7, 148.0)
- added ?: MountingHole_3.5mm, MountingHole:MountingHole_3.5mm, F.Cu at (160.3, 142.5)
- added ?: MountingHole_3.5mm, MountingHole:MountingHole_3.5mm, F.Cu at (89.4, 145.3)
- added ?: MountingHole_3.5mm, MountingHole:MountingHole_3.5mm, F.Cu at (42.0, 148.0)
- added ?: MountingHole_3.5mm, MountingHole:MountingHole_3.5mm, F.Cu at (135.3, 145.3)
- added ?: MountingHole_3.5mm, MountingHole:MountingHole_3.5mm, F.Cu at (135.3, 84.3)
- added C21: C, Capacitor_THT:CP_Radial_D8.0mm_P3.50mm, F.Cu at (48.5, 103.5)
- added REF**: MountingHole_3.5mm, MountingHole:MountingHole_3.5mm, F.Cu at (59.9, 144.3)
- added ZD: 4148, Diode_THT:D_DO-34_SOD68_P7.62mm_Horizontal, F.Cu at (138.9, 117.9)
- C11, C14, C17, C6, C9, R10, R11, R13, R32, R33, R35, R37, R38, R39, R40, R41, R44, R48, R49: moved to B.Cu
- C12: footprint Capacitor_SMD:C_0805_2012Metric_Pad1.15x1.40mm_HandSolder -> Capacitor_THT:C_Disc_D7.5mm_W5.0mm_P7.50mm
- C15: footprint Capacitor_THT:CP_Radial_D22.0mm_P10.00mm_SnapIn -> Capacitor_SMD:C_0805_2012Metric_Pad1.15x1.40mm_HandSolder; moved to B.Cu
- C16: footprint Capacitor_THT:CP_Radial_D14.0mm_P5.00mm -> Capacitor_THT:CP_Radial_D5.0mm_P2.50mm
- C18: footprint Capacitor_THT:CP_Radial_D22.0mm_P10.00mm_3pin_SnapIn -> Capacitor_THT:CP_Radial_D4.0mm_P2.00mm
- C19: footprint Capacitor_THT:CP_Radial_D12.5mm_P2.50mm -> Capacitor_THT:CP_Radial_D12.5mm_P7.50mm
- C20: footprint Capacitor_THT:CP_Radial_D22.0mm_P10.00mm_SnapIn -> Capacitor_THT:CP_Radial_D8.0mm_P3.50mm
- C3: footprint Capacitor_THT:CP_Radial_D22.0mm_P10.00mm_SnapIn -> Capacitor_THT:CP_Radial_D5.0mm_P2.50mm
- C4: footprint Capacitor_THT:CP_Radial_D22.0mm_P10.00mm_SnapIn -> Capacitor_THT:CP_Radial_D10.0mm_P5.00mm_P7.50mm
- C5: footprint Capacitor_THT:CP_Radial_D22.0mm_P10.00mm_SnapIn -> Capacitor_THT:CP_Radial_D10.0mm_P7.50mm
- C7: footprint Capacitor_THT:CP_Radial_D22.0mm_P10.00mm_SnapIn -> Capacitor_SMD:C_0805_2012Metric; moved to B.Cu
- C8: footprint Capacitor_SMD:C_0805_2012Metric_Pad1.15x1.40mm_HandSolder -> Capacitor_THT:CP_Radial_D8.0mm_P5.00mm
- D1, D3, D4: footprint Diode_THT:D_DO-27_P15.24mm_Horizontal -> Diode_THT:D_DO-41_SOD81_P10.16mm_Horizontal
- D6: footprint Diode_THT:D_DO-34_SOD68_P7.62mm_Horizontal -> Diode_THT:D_DO-41_SOD81_P10.16mm_Horizontal
- D8: footprint Diode_THT:D_DO-27_P15.24mm_Horizontal -> Diode_THT:D_DO-201AD_P15.24mm_Horizontal
- J1: value Screw_Terminal_01x03 -> (none); footprint 282834-3:2828343 -> TerminalBlock:TerminalBlock_bornier-3_P5.08mm
- J2: footprint Connector_Molex:Molex_PicoBlade_53047-0610_1x06_P1.25mm_Vertical -> Connector_JST:JST_PH_B6B-PH-K_1x06_P2.00mm_Vertical
- L1, L2: footprint Inductor_THT:L_Radial_D12.0mm_P6.00mm_MuRATA_1900R -> Inductor_THT:L_Radial_D12.0mm_P10.00mm_Neosid_SD12_style1
- LED1, LED2: footprint LED_THT:LED_D5.0mm -> LED_THT:LED_D3.0mm
- R1: footprint Resistor_THT:R_Axial_DIN0414_L11.9mm_D4.5mm_P15.24mm_Horizontal -> Resistor_SMD:R_0805_2012Metric_Pad1.15x1.40mm_HandSolder; moved to B.Cu
- R12: footprint Resistor_SMD:R_0805_2012Metric_Pad1.15x1.40mm_HandSolder -> Resistor_THT:R_Axial_DIN0207_L6.3mm_D2.5mm_P10.16mm_Horizontal
- R14, R16, R17, R18, R20, R27, R28, R29, R45, R46, R47, R5: footprint Resistor_THT:R_Axial_DIN0411_L9.9mm_D3.6mm_P20.32mm_Horizontal -> Resistor_THT:R_Axial_DIN0207_L6.3mm_D2.5mm_P10.16mm_Horizontal
- R15, R7, R8: footprint Resistor_THT:R_Axial_DIN0411_L9.9mm_D3.6mm_P20.32mm_Horizontal -> Resistor_SMD:R_0805_2012Metric_Pad1.15x1.40mm_HandSolder; moved to B.Cu
- R19: footprint Resistor_THT:R_Axial_DIN0411_L9.9mm_D3.6mm_P20.32mm_Horizontal -> Resistor_THT:R_Axial_DIN0309_L9.0mm_D3.2mm_P12.70mm_Horizontal
- R2: footprint Resistor_THT:R_Axial_DIN0516_L15.5mm_D5.0mm_P20.32mm_Horizontal -> Resistor_THT:R_Axial_DIN0411_L9.9mm_D3.6mm_P15.24mm_Horizontal
- R21, R25, R30: footprint Resistor_THT:R_Axial_DIN0411_L9.9mm_D3.6mm_P20.32mm_Horizontal -> Resistor_THT:R_Axial_DIN0204_L3.6mm_D1.6mm_P7.62mm_Horizontal
- R31: footprint Resistor_THT:R_Axial_DIN0411_L9.9mm_D3.6mm_P20.32mm_Horizontal -> Resistor_THT:R_Axial_DIN0207_L6.3mm_D2.5mm_P15.24mm_Horizontal
- R36: footprint Resistor_SMD:R_0805_2012Metric_Pad1.15x1.40mm_HandSolder -> Resistor_THT:R_Axial_DIN0204_L3.6mm_D1.6mm_P7.62mm_Horizontal
- R4: footprint Resistor_THT:R_Axial_DIN0411_L9.9mm_D3.6mm_P20.32mm_Horizontal -> Resistor_THT:R_Axial_DIN0411_L9.9mm_D3.6mm_P15.24mm_Horizontal
- R42: footprint Resistor_SMD:R_1806_4516Metric_Pad1.57x1.80mm_HandSolder -> Resistor_THT:R_Axial_DIN0207_L6.3mm_D2.5mm_P10.16mm_Horizontal
- R6: footprint Resistor_THT:R_Axial_DIN0207_L6.3mm_D2.5mm_P15.24mm_Horizontal -> Resistor_THT:R_Axial_DIN0411_L9.9mm_D3.6mm_P15.24mm_Horizontal
- R9: footprint Resistor_THT:R_Axial_DIN0411_L9.9mm_D3.6mm_P25.40mm_Horizontal -> Resistor_THT:R_Axial_DIN0204_L3.6mm_D1.6mm_P7.62mm_Horizontal
- U6: footprint Package_TO_SOT_THT:TO-220-5_Vertical -> Package_TO_SOT_THT:TO-220-5_P3.4x3.7mm_StaggerOdd_Lead3.8mm_Vertical
- moved C19 204.4 mm to (44.2, 131.1), turned to 45 degrees
- moved LED1 183.9 mm to (52.1, 115.8), turned to 180 degrees
- moved C6 176.5 mm to (45.1, 102.9), turned to 270 degrees
- moved LED2 157.7 mm to (46.2, 89.4), turned to 90 degrees
- moved U4 155.5 mm to (61.5, 82.8), turned to 180 degrees
- moved J2 154.9 mm to (40.6, 95.9), turned to 270 degrees
- moved U3 153.5 mm to (80.0, 85.1), turned to 90 degrees
- moved D6 140.8 mm to (104.8, 102.2), turned to 90 degrees
- moved C17 137.2 mm to (43.4, 92.7), turned to 90 degrees
- moved C16 133.0 mm to (57.1, 90.9)
- moved D2 129.9 mm to (127.3, 117.9)
- moved C1 123.9 mm to (116.2, 133.3), turned to 270 degrees
- moved R12 123.5 mm to (50.5, 92.5), turned to 90 degrees
- moved C5 122.0 mm to (139.4, 135.1), turned to 90 degrees
- moved C12 118.1 mm to (68.6, 87.6), turned to 90 degrees
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Connections:
- C18 pad 1: Net-(C18-Pad1) -> TO_FB1
- T1 pad 14: (no net) -> Net-(C2-Pad2)
- T1 pad 5: Net-(C2-Pad2) -> (no net)
Routing:
- net Earth: track 0.00 -> 656.3 mm
- net Net-(C8-Pad1): track 0.00 -> 128.3 mm
- net OPTO_POS+: track 0.00 -> 109.8 mm
- net OPTO_2: track 0.00 -> 72.3 mm
- net Net-(C1-Pad2): track 0.00 -> 65.1 mm
- net TO_FB1: track 0.00 -> 61.6 mm
- net Net-(C12-Pad2): track 0.00 -> 54.0 mm
- net Net-(C4-Pad1): track 0.00 -> 44.2 mm
- net Net-(C15-Pad2): track 0.00 -> 36.6 mm
- net Net-(Q4-Pad3): track 0.00 -> 32.5 mm
- net Net-(C20-Pad1): track 0.00 -> 31.3 mm
- net 358IN: track 0.00 -> 31.2 mm
- net Net-(D4-Pad1): track 0.00 -> 31.2 mm
- net Net-(C2-Pad2): track 0.00 -> 31.1 mm
- net Net-(R28-Pad1): track 0.00 -> 31.1 mm
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- added copper zone on B.Cu, net 358IN
- added copper zone on B.Cu, net 48V
- added copper zone on B.Cu, net Earth
- added copper zone on B.Cu, net Net-(C1-Pad1)
- added copper zone on B.Cu, net Net-(C1-Pad2)
- added copper zone on B.Cu, net Net-(C2-Pad2)
- added copper zone on B.Cu, net Net-(J1-Pad3)
- added copper zone on B.Cu, net OPTO_2
Other:
- board outline added: 160 x 74.9 mm
- board text added: "-48V+"
- board text added: "-5V+"
- board text added: "INPUT"
- board text added: "MES-2443-01 (480 580 490 171)"
