File: supplyboard/supplyboard.sch (KiCad schematic (older format))
At the start: 95 parts, among them J1 Screw_Terminal_01x03, J2 FEMALE 06, J3 Conn_01x02, Q1 MBR20100CT, Q2 MBR20100CT, Q3 PN2222A, Q4 IRF540N, Q5 PN2222A, T1 SM_FB, U1 EL817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

Commit message: finalgerber
Parts:
- added C21: CP, Capacitor_THT:CP_Radial_D10.0mm_P7.50mm, symbol Device:CP
- C15, C20, C3, C4, C5, C7: footprint Capacitor_THT:CP_Radial_D22.0mm_P10.00mm_SnapIn -> Capacitor_THT:CP_Radial_D10.0mm_P7.50mm
- C18: footprint Capacitor_THT:CP_Radial_D22.0mm_P10.00mm_3pin_SnapIn -> Capacitor_THT:CP_Radial_D10.0mm_P7.50mm
- C19: footprint Capacitor_THT:CP_Radial_D12.5mm_P2.50mm -> Capacitor_THT:CP_Radial_D10.0mm_P7.50mm
- R14, R15, R16, R17, R18, R19, R20, R21, R25, R27, R28, R29, R30, R31, R4, R45, R46, R47, R5, R7, R8: footprint Resistor_THT:R_Axial_DIN0411_L9.9mm_D3.6mm_P20.32mm_Horizontal -> Resistor_THT:R_Axial_DIN0411_L9.9mm_D3.6mm_P12.70mm_Horizontal
- R6: footprint Resistor_THT:R_Axial_DIN0207_L6.3mm_D2.5mm_P15.24mm_Horizontal -> Resistor_THT:R_Axial_DIN0411_L9.9mm_D3.6mm_P12.70mm_Horizontal
- R9: footprint Resistor_THT:R_Axial_DIN0411_L9.9mm_D3.6mm_P25.40mm_Horizontal -> Resistor_THT:R_Axial_DIN0411_L9.9mm_D3.6mm_P12.70mm_Horizontal
Connections:
- net 48V: now also C21.1
- net Earth: now also C21.2
